File: Schematics/Display Driver/Display Driver.kicad_sch (KiCad schematic)
At the start: 108 parts

Commit message: commit
Parts:
- removed D1, D10, D100, D101, D102, D103, D104, D105, D106, D107, D108, D11, D12, D13, D14, D15, D16, D17, D18, D19, D2, D20, D21, D22, D23, D24, D25, D26, D27, D28, D29, D3, D30, D31, D32, D33, D34, D35, D36, D37, D38, D39, D4, D40, D41, D42, D43, D44, D45, D46, D47, D48, D49, D5, D50, D51, D52, D53, D54, D55, D56, D57, D58, D59, D6, D60, D61, D62, D63, D64, D65, D66, D67, D68, D69, D7, D70, D71, D72, D73, D74, D75, D76, D77, D78, D79, D8, D80, D81, D82, D83, D84, D85, D86, D87, D88, D89, D9, D90, D91, D92, D93, D94, D95, D96, D97, D98, D99: LED, symbol Device:LED
- added J1, J2, J3, J4, J5, J6, J7, J8: XH-5A, Connector_JST:JST_XH_B5B-XH-A_1x05_P2.50mm_Vertical, symbol Connector:Conn_01x05_Socket
- added J9: DIN-5, Connector_JST:JST_XH_B5B-XH-A_1x05_P2.50mm_Vertical, symbol Connector:DIN-5
- added Q1, Q10, Q11, Q12, Q13, Q14, Q15, Q16, Q17, Q18, Q19, Q2, Q20, Q21, Q22, Q23, Q24, Q25, Q26, Q27, Q28, Q29, Q3, Q30, Q31, Q32, Q4, Q5, Q6, Q7, Q8, Q9: 2N3904, Package_TO_SOT_THT:TO-92_Inline, symbol Transistor_BJT:2N3904
- added R1, R17, R19, R2, R21, R23, R25, R27, R29, R3, R31, R33, R35, R37, R39, R4, R41, R43, R45, R47, R49, R5, R51, R53, R55, R57, R59, R6, R61, R63, R7, R8: 470, Resistor_THT:R_Axial_DIN0207_L6.3mm_D2.5mm_P10.16mm_Horizontal, symbol Device:R
- added R10, R11, R12, R13, R14, R15, R16, R18, R20, R22, R24, R26, R28, R30, R32, R34, R36, R38, R40, R42, R44, R46, R48, R50, R52, R54, R56, R58, R60, R62, R64, R9: 330, Resistor_THT:R_Axial_DIN0207_L6.3mm_D2.5mm_P10.16mm_Horizontal, symbol Device:R
- added U1, U2, U3, U4: 74HC595, Package_DIP:DIP-16_W7.62mm, symbol 74xx:74HC595
Connections:
- new net: R27.1, U2.5 (QF)
- new net: Q14.2 (B), R27.2
- new net: J8.1 (Pin_1), R58.2
- new net: J8.2 (Pin_2), R60.2
- new net: J8.3 (Pin_3), R62.2
- new net: J8.4 (Pin_4), R64.2
- new net: Q12.3 (C), R24.1
- new net: J3.4 (Pin_4), R24.2
- new net: Q30.3 (C), R60.1
- new net: Q32.2 (B), R63.2
- new net: Q32.3 (C), R64.1
- new net: R37.1, U3.2 (QC)
- new net: Q19.2 (B), R37.2
- new net: Q23.3 (C), R46.1
- new net: J6.3 (Pin_3), R46.2
- new net: R23.1, U2.3 (QD)
- new net: Q12.2 (B), R23.2
- new net: Q7.2 (B), R7.2
- new net: Q7.3 (C), R15.1
- new net: Q30.2 (B), R59.2
- new net: R6.1, U1.5 (QF)
- new net: Q6.2 (B), R6.2
- new net: Q9.3 (C), R18.1
- new net: J3.1 (Pin_1), R18.2
- new net: Q8.3 (C), R16.1
- new net: J2.4 (Pin_4), R16.2
- new net: Q15.2 (B), R29.2
- new net: Q15.3 (C), R30.1
- new net: R3.1, U1.2 (QC)
- new net: Q3.2 (B), R3.2
- new net: R2.1, U1.1 (QB)
- new net: J9.3, U1.11 (SRCLK), U2.11 (SRCLK), U3.11 (SRCLK), U4.11 (SRCLK)
- new net: J9.4, U1.12 (RCLK), U2.12 (RCLK), U3.12 (RCLK), U4.12 (RCLK)
- new net: J9.2, U1.14 (SER)
- new net: R1.1, U1.15 (QA)
- new net: R4.1, U1.3 (QD)
- new net: R5.1, U1.4 (QE)
- new net: R7.1, U1.6 (QG)
- new net: R8.1, U1.7 (QH)
- new net: U1.9 (QH'), U2.14 (SER)
- new net: R59.1, U4.5 (QF)
- new net: Q5.2 (B), R5.2
- new net: R25.1, U2.4 (QE)
- new net: Q13.2 (B), R25.2
- new net: R45.1, U3.6 (QG)
- new net: Q23.2 (B), R45.2
- new net: R21.1, U2.2 (QC)
- new net: Q11.2 (B), R21.2
- new net: R33.1, U3.15 (QA)
- new net: Q17.2 (B), R33.2
- new net: Q31.2 (B), R61.2
- new net: Q31.3 (C), R62.1
- new net: R63.1, U4.7 (QH)
- new net: Q1.3 (C), R9.1
- new net: J1.1 (Pin_1), R9.2
- new net: R35.1, U3.1 (QB)
- new net: U2.9 (QH'), U3.14 (SER)
- new net: R39.1, U3.3 (QD)
- new net: R41.1, U3.4 (QE)
- new net: R43.1, U3.5 (QF)
- new net: R47.1, U3.7 (QH)
- new net: U3.9 (QH'), U4.14 (SER)
- new net: Q1.2 (B), R1.2
- new net: Q16.3 (C), R32.1
- new net: J4.4 (Pin_4), R32.2
- new net: Q10.2 (B), R19.2
- new net: Q10.3 (C), R20.1
- new net: Q6.3 (C), R14.1
- new net: J2.2 (Pin_2), R14.2
- new net: Q3.3 (C), R11.1
- new net: J1.3 (Pin_3), R11.2
- new net: Q14.3 (C), R28.1
- new net: J4.2 (Pin_2), R28.2
- new net: Q20.3 (C), R40.1
- new net: J5.4 (Pin_4), R40.2
- new net: Q16.2 (B), R31.2
- new net: Q5.3 (C), R13.1
- new net: R61.1, U4.6 (QG)
- new net: J1.2 (Pin_2), R10.2
- new net: J1.4 (Pin_4), R12.2
- new net: Q11.3 (C), R22.1
- new net: J7.1 (Pin_1), R50.2
- new net: J7.2 (Pin_2), R52.2
- new net: J7.3 (Pin_3), R54.2
- new net: J7.4 (Pin_4), R56.2
- new net: Q28.2 (B), R55.2
- new net: Q28.3 (C), R56.1
- new net: Q29.3 (C), R58.1
- new net: Q22.2 (B), R43.2
- new net: Q22.3 (C), R44.1
- new net: J2.3 (Pin_3), R15.2
- new net: Q27.3 (C), R54.1
- new net: Q4.2 (B), R4.2
- new net: Q4.3 (C), R12.1
- new net: J5.1 (Pin_1), R34.2
- new net: J5.2 (Pin_2), R36.2
- new net: J5.3 (Pin_3), R38.2
- new net: R29.1, U2.6 (QG)
- new net: J2.1 (Pin_1), R13.2
- new net: Q9.2 (B), R17.2
- new net: Q18.2 (B), R35.2
- new net: Q18.3 (C), R36.1
- new net: J4.3 (Pin_3), R30.2
- new net: Q13.3 (C), R26.1
- new net: J3.3 (Pin_3), R22.2
- new net: R57.1, U4.4 (QE)
- new net: Q29.2 (B), R57.2
- new net: J6.1 (Pin_1), R42.2
- new net: J6.2 (Pin_2), R44.2
- new net: J6.4 (Pin_4), R48.2
- new net: Q2.2 (B), R2.2
- new net: Q2.3 (C), R10.1
- new net: Q26.2 (B), R51.2
- new net: Q26.3 (C), R52.1
- new net: J3.2 (Pin_2), R20.2
- new net: R51.1, U4.1 (QB)
- new net: R49.1, U4.15 (QA)
- new net: R53.1, U4.2 (QC)
- new net: R55.1, U4.3 (QD)
- new net: Q25.2 (B), R49.2
- new net: Q25.3 (C), R50.1
- new net: Q21.2 (B), R41.2
- new net: Q21.3 (C), R42.1
- new net: Q8.2 (B), R8.2
- new net: R19.1, U2.1 (QB)
- new net: R17.1, U2.15 (QA)
- new net: R31.1, U2.7 (QH)
- new net: Q20.2 (B), R39.2
- new net: J4.1 (Pin_1), R26.2
- new net: Q19.3 (C), R38.1
- new net: Q27.2 (B), R53.2
- new net: Q17.3 (C), R34.1
- new net: Q24.2 (B), R47.2
- new net: Q24.3 (C), R48.1
- new net +12V: J1.5 (Pin_5), J2.5 (Pin_5), J3.5 (Pin_5), J4.5 (Pin_5), J5.5 (Pin_5), J6.5 (Pin_5), J7.5 (Pin_5), J8.5 (Pin_5)
- new net +5V: J9.1, U1.10 (~{SRCLR}), U1.16 (VCC), U2.10 (~{SRCLR}), U2.16 (VCC), U3.10 (~{SRCLR}), U3.16 (VCC), U4.10 (~{SRCLR}), U4.16 (VCC)
- new net GND: J9.5, Q1.1 (E), Q10.1 (E), Q11.1 (E), Q12.1 (E), Q13.1 (E), Q15.1 (E), Q16.1 (E), Q17.1 (E), Q18.1 (E), Q19.1 (E), Q2.1 (E), Q20.1 (E), Q21.1 (E), Q23.1 (E), Q24.1 (E), Q25.1 (E), Q26.1 (E), Q27.1 (E), Q28.1 (E), Q29.1 (E), Q3.1 (E), Q31.1 (E), Q32.1 (E), Q4.1 (E), Q5.1 (E), Q7.1 (E), Q8.1 (E), Q9.1 (E), U1.13 (~{OE}), U1.8 (GND), U2.13 (~{OE}), U2.8 (GND), U3.13 (~{OE}), U3.8 (GND), U4.13 (~{OE}), U4.8 (GND)
